File: pcb.sch (KiCad schematic (older format))
At the start: 36 parts, among them J1 TYPE-C-31-M-12, Q1 FDN339AN, SW1 SW_SPST, U1 WeMos_D1_mini, U2 TSOP38236, U3 MCP73831-2-OT, U4 BQ27441DRZR-G1A, U5 TLV75733PDBV

Commit message: Implemented on-board cell protection to allow the use of un-protected cells
Parts:
- removed BT1: protected 18650, Battery:BatteryHolder_Keystone_1042_1x18650, symbol Device:Battery_Cell
- removed C1: 1uF, Capacitor_SMD:C_0603_1608Metric_Pad1.05x0.95mm_HandSolder, symbol Device:C_Small
- removed C2, C5, C6: 4.7uF, Capacitor_SMD:C_0805_2012Metric_Pad1.15x1.40mm_HandSolder, symbol Device:C_Small
- removed C3, C4: 10nF, Capacitor_SMD:C_0603_1608Metric_Pad1.05x0.95mm_HandSolder, symbol Device:C_Small
- removed D1, D3: VSML3710-GS18, LED_SMD:LED_PLCC-2, symbol Device:LED_Small
- removed D2: BAT54WS, Diode_SMD:D_SOD-323_HandSoldering, symbol Device:D_Schottky_Small
- removed D4: MBRA140, Diode_SMD:D_SMA, symbol Device:D_Schottky_Small
- removed D5: charging, LED_SMD:LED_0603_1608Metric_Pad1.05x0.95mm_HandSolder, symbol Device:LED_Small
- removed D6: charged, LED_SMD:LED_0603_1608Metric_Pad1.05x0.95mm_HandSolder, symbol Device:LED_Small
- removed J1: TYPE-C-31-M-12, Connector_USB:USB_C_Receptacle_HRO_TYPE-C-31-M-12, symbol Connector:USB_C_Receptacle_USB2.0
- removed Q1: FDN339AN, Package_TO_SOT_SMD:SOT-23_Handsoldering, symbol Device:Q_NMOS_GSD
- removed R1, R5, R6: 4k7, Resistor_SMD:R_0603_1608Metric_Pad1.05x0.95mm_HandSolder, symbol Device:R_Small
- removed R10, R14, R15, R4: 10k, Resistor_SMD:R_0603_1608Metric_Pad1.05x0.95mm_HandSolder, symbol Device:R_Small
- removed R11, R12: 470R, Resistor_SMD:R_0603_1608Metric_Pad1.05x0.95mm_HandSolder, symbol Device:R_Small
- removed R13: 10mR, Resistor_SMD:R_0603_1608Metric_Pad1.05x0.95mm_HandSolder, symbol Device:R_Small
- removed R2: 1k, Resistor_SMD:R_0603_1608Metric_Pad1.05x0.95mm_HandSolder, symbol Device:R_Small
- removed R3, R7: 6R8, Resistor_SMD:R_0603_1608Metric_Pad1.05x0.95mm_HandSolder, symbol Device:R_Small
- removed R8, R9: 5k1, Resistor_SMD:R_0603_1608Metric_Pad1.05x0.95mm_HandSolder, symbol Device:R_Small
- removed SW1: SW_SPST, Button_Switch_SMD:SW_Push_1P1T_NO_6x6mm_H9.5mm, symbol Switch:SW_SPST
- removed U1: WeMos_D1_mini, Module:WEMOS_D1_mini_light, symbol MCU_Module:WeMos_D1_mini
- removed U2: TSOP38236, OptoDevice:Vishay_MINICAST-3Pin, symbol Interface_Optical:TSOP382xx
- removed U3: MCP73831-2-OT, Package_TO_SOT_SMD:SOT-23-5, symbol Battery_Management:MCP73831-2-OT
- removed U4: BQ27441DRZR-G1A, Package_SON:Texas_S-PDSO-N12, symbol Battery_Management:BQ27441DRZR-G1A
- removed U5: TLV75733PDBV, Package_TO_SOT_SMD:SOT-23-5, symbol Regulator_Linear:TLV75733PDBV
- added U3: LC709203FQH-01TWG, Package_DFN_QFN:WDFN-8-1EP_4x3mm_P0.65mm_EP2.4x1.8mm, symbol Battery_Management:LC709203FQH-01TWG
Connections:
- net labels removed: +1V8, +BATT, GND, IR_BLAST, IR_RECV_VCC, IR_SIGNAL, SCL, SDA, VBUS, VCCQ, device_wake, factory_rst, ~LOW_BAT, ~RST
- wire segments 113 -> 5
Other:
- note added: "Alternative, cheaper fuel gauge (with no current sense)"
- note removed: "3V3 LDO"
- note removed: "Charging"
- note removed: "Fuel gauge"
- note removed: "IR"
- note removed: "Logic"
- note removed: "MCU"
- note removed: "Power"
- note removed: "Reset circuit"
