File: pcb.kicad_sch (KiCad schematic)
At the start: 31 parts, among them J1 4.5-18V, Q1 FDN339AN, SW1 SW_SPST, U1 WeMos_D1_mini, U2 TSOP38236, U3 TPS54302, U4 AP131-18, U5 SGP30, U6 AHT20

Commit message: v0.4 production
Parts:
- R10, R2: renamed from R?; value 5k1 -> 4k7
- R3, R4: value 5k1 -> 4k7
- R6: value 1k -> 470R
- gave numbers to parts that had none: 2
Connections:
- net VBUS renamed VCC
Changed lines of the file:
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@@
     (pin "1")
   )
-  (symbol (lib_id "power:VBUS") (at 62.865 36.195 0) (unit 1)
-    (in_bom yes) (on_board yes)
-    (property "Reference" "#PWR0110" (id 0) (at 62.865 40.005 0)
-      (effects (font (size 1.27 1.27)) hide)
-    )
-    (property "Value" "VBUS" (id 1) (at 63.246 31.8008 0))
+  (symbol (lib_id "power:VCC") (at 62.865 36.195 0) (unit 1)
+    (in_bom yes) (on_board yes)
+    (property "Reference" "#PWR?" (id 0) (at 62.865 40.005 0)
+      (effects (font (size 1.27 1.27)) hide)
+    )
+    (property "Value" "VCC" (id 1) (at 64.135 30.48 0))
     (property "Footprint" "" (id 2) (at 62.865 36.195 0)
       (effects (font (size 1.27 1.27)) hide)
@@
   (symbol (lib_id "power:+3V3") (at 160.655 104.14 0) (unit 1)
     (in_bom yes) (on_board yes)
-    (property "Reference" "#PWR?" (id 0) (at 160.655 107.95 0)
+    (property "Reference" "#PWR0120" (id 0) (at 160.655 107.95 0)
       (effects (font (size 1.27 1.27)) hide)
     )
@@
     (pin "1")
   )
-  (symbol (lib_id "power:VBUS") (at 222.25 36.195 0) (unit 1)
-    (in_bom yes) (on_board yes)
-    (property "Reference" "#PWR0101" (id 0) (at 222.25 40.005 0)
-      (effects (font (size 1.27 1.27)) hide)
-    )
-    (property "Value" "VBUS" (id 1) (at 222.631 31.8008 0))
+  (symbol (lib_id "power:VCC") (at 222.25 36.195 0) (unit 1)
+    (in_bom yes) (on_board yes)
+    (property "Reference" "#PWR?" (id 0) (at 222.25 40.005 0)
+      (effects (font (size 1.27 1.27)) hide)
+    )
+    (property "Value" "VCC" (id 1) (at 223.52 30.48 0))
     (property "Footprint" "" (id 2) (at 222.25 36.195 0)
       (effects (font (size 1.27 1.27)) hide)
@@
   (symbol (lib_id "power:GND") (at 163.195 132.08 0) (unit 1)
     (in_bom yes) (on_board yes)
-    (property "Reference" "#PWR?" (id 0) (at 163.195 138.43 0)
+    (property "Reference" "#PWR0121" (id 0) (at 163.195 138.43 0)
       (effects (font (size 1.27 1.27)) hide)
     )
@@
   (symbol (lib_id "Device:R_Small") (at 151.765 113.03 0) (mirror x) (unit 1)
     (in_bom yes) (on_board yes)
-    (property "Reference" "R?" (id 0) (at 150.2664 111.8616 0)
+    (property "Reference" "R1" (id 0) (at 150.2664 111.8616 0)
       (effects (font (size 1.27 1.27)) (justify right))
     )
@@
       (effects (font (size 1.27 1.27)) (justify right))
     )
-    (property "Value" "5k1" (id 1) (at 175.6664 43.053 0)
+    (property "Value" "4k7" (id 1) (at 175.666 43.053 0)
       (effects (font (size 1.27 1.27)) (justify right))
     )
@@
   (symbol (lib_id "Device:R_Small") (at 177.165 114.935 0) (mirror x) (unit 1)
     (in_bom yes) (on_board yes)
-    (property "Reference" "R?" (id 0) (at 175.6664 113.7666 0)
-      (effects (font (size 1.27 1.27)) (justify right))
-    )
-    (property "Value" "5k1" (id 1) (at 175.6664 116.078 0)
+    (property "Reference" "R2" (id 0) (at 175.6664 113.7666 0)
+      (effects (font (size 1.27 1.27)) (justify right))
+    )
+    (property "Value" "4k7" (id 1) (at 175.666 116.078 0)
       (effects (font (size 1.27 1.27)) (justify right))
     )
@@
       (effects (font (size 1.27 1.27)) (justify right))
     )
-    (property "Value" "5k1" (id 1) (at 181.204 43.053 0)
+    (property "Value" "4k7" (id 1) (at 181.204 43.053 0)
       (effects (font (size 1.27 1.27)) (justify right))
     )
@@
   (symbol (lib_id "Device:R_Small") (at 179.705 114.935 180) (unit 1)
     (in_bom yes) (on_board yes)
-    (property "Reference" "R?" (id 0) (at 181.2036 113.7666 0)
-      (effects (font (size 1.27 1.27)) (justify right))
-    )
-    (property "Value" "5k1" (id 1) (at 181.2036 116.078 0)
+    (property "Reference" "R10" (id 0) (at 181.2036 113.7666 0)
+      (effects (font (size 1.27 1.27)) (justify right))
+    )
+    (property "Value" "4k7" (id 1) (at 181.204 116.078 0)
       (effects (font (size 1.27 1.27)) (justify right))
     )
@@
       (effects (font (size 1.27 1.27)) (justify right))
     )
-    (property "Value" "4k7" (id 1) (at 206.7814 67.183 0)
+    (property "Value" "4k7" (id 1) (at 206.781 67.183 0)
       (effects (font (size 1.27 1.27)) (justify right))
     )
@@
     (in_bom yes) (on_board yes)
     (property "Reference" "R6" (id 0) (at 212.09 57.2516 90))
-    (property "Value" "1k" (id 1) (at 212.09 59.563 90))
+    (property "Value" "470R" (id 1) (at 212.09 59.563 90))
     (property "Footprint" "Resistor_SMD:R_0603_1608Metric_Pad0.98x0.95mm_HandSolder" (id 2) (at 212.09 62.23 0)
       (effects (font (size 1.27 1.27)) hide)
@@
       (effects (font (size 1.27 1.27)) hide)
     )
-    (property "MPN" "CL10A226MP8NUNE" (id 4) (at 115.57 54.61 0))
+    (property "MPN" "CL10A226MP8NUNE" (id 4) (at 116.84 55.88 0))
     (pin "1")
     (pin "2")
@@
   (symbol (lib_id "Interface:PCA9306DC1") (at 163.195 119.38 0) (mirror y) (unit 1)
     (in_bom yes) (on_board yes)
-    (property "Reference" "U?" (id 0) (at 157.48 130.81 0))
+    (property "Reference" "U7" (id 0) (at 157.48 130.81 0))
     (property "Value" "PCA9306DC1" (id 1) (at 170.18 130.81 0))
     (property "Footprint" "Package_SO:VSSOP-8_2.3x2mm_P0.5mm" (id 2) (at 163.195 130.81 0)
@@
   )
   (symbol_instances
-    (path "/58115fe6-543f-4dc3-8e0c-854290afdcd8"
-      (reference "#PWR0101") (unit 1) (value "VBUS") (footprint "")
-    )
     (path "/4bdefbc2-e60e-45e3-b469-c7e4ee78db2b"
       (reference "#PWR0102") (unit 1) (value "GND") (footprint "")
@@
       (reference "#PWR0109") (unit 1) (value "GND") (footprint "")
     )
-    (path "/90d731b8-177f-47e5-a5ff-52f6243ff053"
-      (reference "#PWR0110") (unit 1) (value "VBUS") (footprint "")
-    )
     (path "/5c7c2a79-b84f-4834-8ff5-1c86de6fbb47"
       (reference "#PWR0111") (unit 1) (value "GND") (footprint "")
@@
       (reference "#PWR0119") (unit 1) (value "+3V3") (footprint "")
     )
+    (path "/7d59b3a0-8f47-40c3-86ee-962d0aa72dd9"
+      (reference "#PWR0120") (unit 1) (value "+3V3") (footprint "")
+    )
     (path "/6c1def17-6701-42eb-9ba1-f5d73c983607"
-      (reference "#PWR?") (unit 1) (value "GND") (footprint "")
-    )
-    (path "/7d59b3a0-8f47-40c3-86ee-962d0aa72dd9"
-      (reference "#PWR?") (unit 1) (value "+3V3") (footprint "")
+      (reference "#PWR0121") (unit 1) (value "GND") (footprint "")
+    )
+    (path "/93354151-6a49-40a1-8659-7b7979c22e83"
+      (reference "#PWR?") (unit 1) (value "VCC") (footprint "")
+    )
+    (path "/d700b45b-bf50-4ed3-8e15-645fe836c13b"
+      (reference "#PWR?") (unit 1) (value "VCC") (footprint "")
     )
     (path "/3e5bf149-c738-4d8c-98c7-60805c47a399"
@@
       (reference "Q1") (unit 1) (value "FDN339AN") (footprint "Package_TO_SOT_SMD:SOT-23_Handsoldering")
     )
+    (path "/e5579559-ce37-4749-89a9-1062775b5c94"
+      (reference "R1") (unit 1) (value "22k") (footprint "Resistor_SMD:R_0603_1608Metric_Pad0.98x0.95mm_HandSolder")
+    )
+    (path "/0b48628e-b3e8-4d9c-b889-835fd1762803"
+      (reference "R2") (unit 1) (value "4k7") (footprint "Resistor_SMD:R_0603_1608Metric_Pad0.98x0.95mm_HandSolder")
+    )
     (path "/2fb37f15-cfd9-452c-a896-0627c3d35cfa"
-      (reference "R3") (unit 1) (value "5k1") (footprint "Resistor_SMD:R_0603_1608Metric_Pad0.98x0.95mm_HandSolder")
+      (reference "R3") (unit 1) (value "4k7") (footprint "Resistor_SMD:R_0603_1608Metric_Pad0.98x0.95mm_HandSolder")
     )
     (path "/e1d36cf1-8d79-4a6e-92bb-6fd16804dfc2"
-      (reference "R4") (unit 1) (value "5k1") (footprint "Resistor_SMD:R_0603_1608Metric_Pad0.98x0.95mm_HandSolder")
+      (reference "R4") (unit 1) (value "4k7") (footprint "Resistor_SMD:R_0603_1608Metric_Pad0.98x0.95mm_HandSolder")
     )
     (path "/c7b6571a-1a14-4fa8-b1c9-4aece29082a2"
@@
     )
     (path "/f906bf8a-aa15-4246-b473-eddd0ec562c0"
-      (reference "R6") (unit 1) (value "1k") (footprint "Resistor_SMD:R_0603_1608Metric_Pad0.98x0.95mm_HandSolder")
+      (reference "R6") (unit 1) (value "470R") (footprint "Resistor_SMD:R_0603_1608Metric_Pad0.98x0.95mm_HandSolder")
     )
     (path "/6b60f39f-1592-4911-be42-25f9f1f2d389"
@@
       (reference "R9") (unit 1) (value "22k") (footprint "Resistor_SMD:R_0603_1608Metric_Pad0.98x0.95mm_HandSolder")
     )
-    (path "/0b48628e-b3e8-4d9c-b889-835fd1762803"
-      (reference "R?") (unit 1) (value "5k1") (footprint "Resistor_SMD:R_0603_1608Metric_Pad0.98x0.95mm_HandSolder")
-    )
     (path "/5dca8f7e-f8a5-4a22-97dd-ff9e335f6469"
-      (reference "R?") (unit 1) (value "5k1") (footprint "Resistor_SMD:R_0603_1608Metric_Pad0.98x0.95mm_HandSolder")
-    )
-    (path "/e5579559-ce37-4749-89a9-1062775b5c94"
-      (reference "R?") (unit 1) (value "22k") (footprint "Resistor_SMD:R_0603_1608Metric_Pad0.98x0.95mm_HandSolder")
+      (reference "R10") (unit 1) (value "4k7") (footprint "Resistor_SMD:R_0603_1608Metric_Pad0.98x0.95mm_HandSolder")
     )
     (path "/1d7e27c6-6983-46cf-90f6-7c7cc5c47f35"
@@
     )
     (path "/5ee4da8f-4281-43fb-a568-902173be53e7"
-      (reference "U?") (unit 1) (value "PCA9306DC1") (footprint "Package_SO:VSSOP-8_2.3x2mm_P0.5mm")
-    )
-  )
+      (reference "U7") (unit 1) (value "PCA9306DC1") (footprint "Package_SO:VSSOP-8_2.3x2mm_P0.5mm")
+    )
+  )

Commit message: Use 220uH inductor and emitter follower LED driver
Parts:
- removed D1, D2: VSML3710-GS18, LED_SMD:LED_PLCC-2, symbol Device:LED_Small
- removed Q1: FDN339AN, Package_TO_SOT_SMD:SOT-23_Handsoldering, symbol Device:Q_NMOS_GSD
- removed R5: 4k7, Resistor_SMD:R_0603_1608Metric_Pad0.98x0.95mm_HandSolder, symbol Device:R_Small
- removed R6: 470R, Resistor_SMD:R_0603_1608Metric_Pad0.98x0.95mm_HandSolder, symbol Device:R_Small
- added D? (x2): VSML3710-GS18, LED_SMD:LED_PLCC-2, symbol Device:LED_Small
- added JP1: 1v8-bp, Jumper:SolderJumper-2_P1.3mm_Open_TrianglePad1.0x1.5mm, symbol Jumper:Jumper_2_Open
- added JP2: sda-bp, Jumper:SolderJumper-2_P1.3mm_Open_TrianglePad1.0x1.5mm, symbol Jumper:Jumper_2_Open
- added JP3: scl-bp, Jumper:SolderJumper-2_P1.3mm_Open_TrianglePad1.0x1.5mm, symbol Jumper:Jumper_2_Open
- added Q?: SS8050, symbol Device:Q_NPN_BEC
- added R?: 5.6R, Resistor_SMD:R_0805_2012Metric_Pad1.20x1.40mm_HandSolder, symbol Device:R_Small
- C5: MPN CL10A226MP8NUNE -> CL21A226MAYNNNE
- J1: value 4.5-18V -> 12V
- L1: value 6.8uH -> 100μH; footprint Inductor_SMD:L_6.3x6.3_H3 -> Inductor_SMD:L_Bourns_SRN6045TA; MPN SLO0530H6R8MTT -> SRN6045-101M
- R7: value 27R -> 5.6R; footprint Resistor_SMD:R_0603_1608Metric_Pad0.98x0.95mm_HandSolder -> Resistor_SMD:R_0805_2012Metric_Pad1.20x1.40mm_HandSolder
Connections:
- net +1V8: now also JP1.1 (A)
- net +3V3: now also JP1.2 (B)
- net GND: now also R7.2, R?.2
- net IR_BLAST: now also Q?.1 (B)
- net IR_SIGNAL: now also U1.4 (SCK/D5); no longer U1.11 (D4)
- net SCL_1V8: now also JP2.1 (A)
- net SCL_3V3: now also JP2.2 (B)
- net SDA_1V8: now also JP3.1 (A)
- net SDA_3V3: now also JP3.2 (B)
- net VCC: now also Q?.3 (C)
- net at R7.1: now also D?.1 (K)
- new net: D?.2 (A), D?.2 (A), Q?.2 (E)
- new net: D?.1 (K), R?.1
Other:
- note added: "1V8 to 3V3 bypass"
- moved on the sheet: R7, U2
